File: PCB/V7/Air Conditioner Energy Saver V7.kicad_sch (KiCad schematic)
At the start: 73 parts, among them J1 Conn_01x05_Male, J2 Conn_01x06_Male, J4 Conn_01x04_Male, J5 Conn_01x04_Male, P13 TestPoint, P16 TestPoint, P17 TestPoint, P2 TestPoint, P22 TestPoint, P23 TestPoint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

Commit message: Updating to the latest V7 PCB that was submitted to JLCPCB
Parts:
- C1, C4: LCSC (none) -> C15195; MN (none) -> Samsung Electro-Mechanics; MPN (none) -> CL05B103KB5NNNC
- C12, C21, C9: LCSC (none) -> C13585; MN (none) -> Samsung Electro-Mechanics; MPN (none) -> CL31A106KBHNNNE
- C14: LCSC (none) -> C282065; MN (none) -> YAGEO; MPN (none) -> CC0603KRX7R9BB203
- C15: LCSC (none) -> C1779; MN (none) -> Samsung Electro-Mechanics; MPN (none) -> CL21A475KAQNNNE
- C16: LCSC (none) -> C15849; MN (none) -> Samsung Electro-Mechanics; MPN (none) -> CL10A105KB8NNNC
- C18, C19, C23: LCSC (none) -> C307331; MN (none) -> Samsung Electro-Mechanics; MPN (none) -> CL05B104KB54PNC
- C2: LCSC (none) -> C19666; MN (none) -> Samsung Electro-Mechanics; MPN (none) -> CL10A475KO8NNNC
- C3: LCSC (none) -> C12891; MN (none) -> Samsung Electro-Mechanics; MPN (none) -> CL31A226KAHNNNE
- C5: MN (none) -> ROQANG; MPN (none) -> RVT1A102M0810
- D1: MN (none) -> Everlight Elec; MPN (none) -> IR333-A
- D3: LCSC (none) -> C108793; MN (none) -> Foshan NationStar Optoelectronics; MPN (none) -> FM-B2020RGBA-HG
- J1: LCSC (none) -> C492404; MN (none) -> XFCN; MPN (none) -> PZ254V-11-05P
- J2: LCSC (none) -> C492405; MN (none) -> XFCN; MPN (none) -> PZ254V-11-06P
- J4, J5: LCSC (none) -> C2691448; MN (none) -> XFCN; MPN (none) -> PZ254V-11-04P
- JP1: LCSC (none) -> C2937625; MN (none) -> XFCN; MPN (none) -> PZ254V-11-03P
- L2: LCSC (none) -> C27143; MN (none) -> Sunlord; MPN (none) -> SDCL1005C15NJTDF
- L3: LCSC (none) -> C1035; MN (none) -> Sunlord; MPN (none) -> SDFL1608S100KTF
- Q1: LCSC (none) -> C85078; MN (none) -> ST(Semtech); MPN (none) -> BC817-40
- Q2: LCSC (none) -> C15127; MN (none) -> Alpha & Omega Semicon; MPN (none) -> AO3401A
- R1: LCSC (none) -> C25900; MN (none) -> UNI-ROYAL(Uniroyal Elec); MPN (none) -> 0402WGF4701TCE
- R10: LCSC (none) -> C138008; MN (none) -> YAGEO; MPN (none) -> RC0402FR-0730KL
- R11, R23, R24, R8: LCSC (none) -> C25744; MN (none) -> UNI-ROYAL(Uniroyal Elec); MPN (none) -> 0402WGF1002TCE
- R12: LCSC (none) -> C25790; MN (none) -> UNI-ROYAL(Uniroyal Elec); MPN (none) -> 0402WGF4703TCE
- R13: LCSC (none) -> C25774; MN (none) -> UNI-ROYAL(Uniroyal Elec); MPN (none) -> 0402WGF3003TCE
- R14: LCSC (none) -> C26083; MN (none) -> UNI-ROYAL(Uniroyal Elec); MPN (none) -> 0402WGF1004TCE
- R15: LCSC (none) -> C23345; MN (none) -> UNI-ROYAL(Uniroyal Elec); MPN (none) -> 0603WAF220JT5E
- R16, R7: LCSC (none) -> C25792; MN (none) -> UNI-ROYAL(Uniroyal Elec); MPN (none) -> 0402WGF4702TCE
- R19, R22: LCSC (none) -> C17168; MN (none) -> UNI-ROYAL(Uniroyal Elec); MPN (none) -> 0402WGF0000TCE
- R2: LCSC (none) -> C23162; MN (none) -> UNI-ROYAL(Uniroyal Elec); MPN (none) -> 0603WAF4701T5E
- R3, R4, R5: LCSC (none) -> C11702; MN (none) -> UNI-ROYAL(Uniroyal Elec); MPN (none) -> 0402WGF1001TCE
- R6: LCSC (none) -> C25537; MN (none) -> UNI-ROYAL(Uniroyal Elec); MPN (none) -> 0402WGJ0133TCE
- R9: LCSC (none) -> C482785; MN (none) -> YAGEO; MPN (none) -> RC0603FR-072M1L
- RST1, RST2, SW1, SW11, SW2, SW22: LCSC (none) -> C720477; MN (none) -> XUNPU; MPN (none) -> TS-1088-AR02016
- U1: MN (none) -> Everlight Elec; MPN (none) -> IRM-H638T/TR2
- U2: MN (none) -> NEWOPTO; MPN (none) -> PIR203A-S0
- U3: MN (none) -> Jiangsu RUNIC Tech; MPN (none) -> RS8032XK
- U3: LCSC (none) -> C237005; MN (none) -> Jiangsu RUNIC Tech; MPN (none) -> RS8032XK
- U4: value E73-2G4M04S-52810 -> E73-2G4M04S1A; LCSC (none) -> C411305; MN (none) -> Chengdu Ebyte Elec Tech; MPN (none) -> E73-2G4M04S1B
- U5: LCSC C259233 -> C259572; MN (none) -> Holtek Semicon; MPN (none) -> HT7218
Connections:
- no-connect marks 3 -> 4
